Commit message: gazebo test world working

File: f1tenth_description/urdf/racecar.xacro (robot description, xacro)
@@ -1,220 +1,62 @@
 <?xml version="1.0"?>
 <robot name="racecar" xmlns:xacro="http://www.ros.org/wiki/xacro">
-  <xacro:include filename="$(find f1tenth_description)/urdf/macros.xacro" />
-  <link name="base_link" />
-  <link name="chassis">
-    <visual>
-      <xacro:chassis_geometry/>
-      <material name="blue" />
-    </visual>
-  </link>
+  <!-- Include macros and materials -->
+  <xacro:include filename="$(find f1tenth_description)/urdf/macros.xacro"/>
+  <xacro:include filename="$(find f1tenth_description)/urdf/materials.xacro"/>
+  <!-- Chassis -->
+  <link name="chassis"/>
+  <link name="base_link"/>
   <joint name="base_link_joint" type="fixed">
-    <origin xyz="0 0 0.05" rpy="0 0 0" />
-    <parent link="base_link" />
-    <child link="chassis" />
+    <parent link="base_link"/>
+    <child link="chassis"/>
+    <origin xyz="0 0 0.05" rpy="0 0 0"/>
   </joint>
-  <link name="chassis_inertia">
-    <inertial>
-      <xacro:chassis_inertial_params />
-    </inertial>
-  </link>
-  <joint name="chassis_inertia_joint" type="fixed">
-    <origin xyz="0 0 0" rpy="0 0 0" />
-    <parent link="chassis" />
-    <child link="chassis_inertia" />
+  <!-- Rear Wheels -->
+  <link name="left_rear_wheel"/>
+  <link name="right_rear_wheel"/>
+  <joint name="left_rear_wheel_joint" type="continuous">
+    <parent link="chassis"/>
+    <child link="left_rear_wheel"/>
+    <axis xyz="0 0 -1"/>
   </joint>
-  <link name="left_rear_wheel">
-    <inertial>
-      <xacro:left_wheels_inertial_params />
-    </inertial>
-    <visual>
-      <xacro:left_rear_wheel_geometry />
-      <material name="black" />
-    </visual>
-    <collision>robot
-      <xacro:left_wheels_collision_geometry />
-    </collision>
-  </link>
-  <joint name="left_rear_wheel_joint" type="continuous">
-    <origin xyz="0 0.1 0" rpy="1.5708 0 0" />
-    <parent link="chassis" />
-    <child link="left_rear_wheel" />
-    <axis xyz="0 0 -1" />
-    <limit effort="10" velocity="100" />
+  <joint name="right_rear_wheel_joint" type="continuous">
+    <parent link="chassis"/>
+    <child link="right_rear_wheel"/>
+    <axis xyz="0 0 -1"/>
   </joint>
-  <xacro:wheel_transmission name="left_rear_wheel" />
-  <link name="right_rear_wheel">
-    <inertial>
-      <xacro:right_wheels_inertial_params />
-    </inertial>
-    <visual>
-      <xacro:right_rear_wheel_geometry />
-      <material name="black" />
-    </visual>
-    <collision>
-      <xacro:right_wheels_collision_geometry />
-    </collision>
-  </link>
-  <joint name="right_rear_wheel_joint" type="continuous">
-    <origin xyz="0 -0.1 0" rpy="1.5708 0 0" />
-    <parent link="chassis" />
-    <child link="right_rear_wheel" />
-    <axis xyz="0 0 -1" />
-    <limit effort="10" velocity="100" />
+  <!-- Steering Hinges -->
+  <link name="left_steering_hinge"/>
+  <link name="right_steering_hinge"/>
+  <joint name="left_steering_hinge_joint" type="revolute">
+    <parent link="chassis"/>
+    <child link="left_steering_hinge"/>
+    <axis xyz="-1 0 0"/>
+    <limit lower="-1.0" upper="1.0"/>
   </joint>
-  <xacro:wheel_transmission name="right_rear_wheel" />
-  <link name="left_steering_hinge">
-    <inertial>
-      <xacro:steering_hinge_inertial_params />
-    </inertial>
-    <visual>
-      <xacro:left_steering_hinge_geometry />
-      <material name="grey" />
-    </visual>
-  </link>
-  <joint name="left_steering_hinge_joint" type="revolute">
-    <origin xyz="0.325 0.1 0" rpy="0 1.5708 0" />
-    <parent link="chassis" />
-    <child link="left_steering_hinge" />
-    <axis xyz="-1 0 0" />
-    <limit lower="-1.0" upper="1.0" effort="10" velocity="100" />
+  <joint name="right_steering_hinge_joint" type="revolute">
+    <parent link="chassis"/>
+    <child link="right_steering_hinge"/>
+    <axis xyz="-1 0 0"/>
+    <limit lower="-1.0" upper="1.0"/>
   </joint>
-  <xacro:steering_hinge_transmission name="left_steering_hinge" />
-  <link name="right_steering_hinge">
-    <inertial>
-      <xacro:steering_hinge_inertial_params />
-    </inertial>
-    <visual>
-      <xacro:right_steering_hinge_geometry />
-      <material name="grey" />
-    </visual>
-  </link>
-  <joint name="right_steering_hinge_joint" type="continuous">
-    <origin xyz="0.325 -0.1 0" rpy="0 1.5708 0" />
-    <parent link="chassis" />
-    <child link="right_steering_hinge" />
-    <axis xyz="-1 0 0" />
-    <limit lower="-1.0" upper="1.0" effort="10" velocity="100" />
+  <!-- Front Wheels -->
+  <link name="left_front_wheel"/>
+  <link name="right_front_wheel"/>
+  <joint name="left_front_wheel_joint" type="continuous">
+    <parent link="left_steering_hinge"/>
+    <child link="left_front_wheel"/>
+    <axis xyz="0 0 -1"/>
   </joint>
-  <xacro:steering_hinge_transmission name="right_steering_hinge" />
-  <link name="left_front_wheel">
-    <inertial>
-      <xacro:left_wheels_inertial_params />
-    </inertial>
-    <visual>
-      <xacro:left_front_wheel_geometry />
-      <material name="black" />
-    </visual>
-    <collision>
-      <xacro:left_wheels_collision_geometry />
-    </collision>
-  </link>
-  <joint name="left_front_wheel_joint" type="continuous">
-    <origin xyz="0 0 0" rpy="1.5708 0 0" />
-    <parent link="left_steering_hinge" />
-    <child link="left_front_wheel" />
-    <axis xyz="0 0 -1" />
-    <limit effort="10" velocity="100" />
+  <joint name="right_front_wheel_joint" type="continuous">
+    <parent link="right_steering_hinge"/>
+    <child link="right_front_wheel"/>
+    <axis xyz="0 0 -1"/>
   </joint>
-  <xacro:wheel_transmission name="left_front_wheel" />
-  <link name="right_front_wheel">
-    <inertial>
-      <xacro:right_wheels_inertial_params />
-    </inertial>
-    <visual>
-      <xacro:right_front_wheel_geometry />
-      <material name="black" />
-    </visual>
-    <collision>
-      <xacro:right_wheels_collision_geometry />
-    </collision>
-  </link>
-  <joint name="right_front_wheel_joint" type="continuous">
-    <origin xyz="0 0 0" rpy="1.5708 0 0" />
-    <parent link="right_steering_hinge" />
-    <child link="right_front_wheel" />
-    <axis xyz="0 0 -1" />
-    <limit effort="10" velocity="100"/>
-  </joint>
-  <xacro:wheel_transmission name="right_front_wheel" />
-  <link name="laser">
-    <inertial>
-      <xacro:hokuyo_inertial_params />
-    </inertial>
-    <collision>
-      <origin xyz="0 0 0" rpy="0 0 0"/>
-      <geometry>
-        <box size="0.1 0.1 0.1"/>
-      </geometry>
-    </collision>
-    <visual>
-      <origin xyz="0 0 0" rpy="0 0 0"/>
-      <geometry>
-        <mesh filename="package://f1tenth_description/meshes/hokuyo.dae"/>
-        <material name="grey" />
-      </geometry>
-    </visual>
-  </link>
-  <joint name="hokuyo_joint" type="fixed">
-    <origin xyz="0.265 0.0 0.075" rpy="0 0 0"/>
-    <parent link="chassis" />
-    <child link="laser" />
-    <axis xyz="0 0 1" />
-  </joint>
-  <link name="zed_camera_link">
-    <inertial>
-      <mass value="1e-5" />
-      <origin xyz="0 0 0" rpy="0 0 0"/>
-      <inertia ixx="1e-6" ixy="0" ixz="0" iyy="1e-6" iyz="0" izz="1e-6" />
-    </inertial>
-    <collision>
-      <origin xyz="0 0 0" rpy="0 0 0"/>
-      <geometry>
-        <box size="0.033 0.175 0.030"/>
-      </geometry>
-    </collision>
-    <visual>
-      <origin xyz="0 0 0" rpy="0 0 0"/>
-      <geometry>
-        <box size="0.033 0.175 0.030"/>
-      </geometry>
-      <material name="red"/>
-    </visual>
-  </link>
-  <joint name="zed_camera_joint" type="fixed">
-    <origin xyz="0.390 0 0.04" rpy="0 0 0"/>
-    <parent link="chassis"/>
-    <child link="zed_camera_link"/>
-    <axis xyz="0 0 1" />
-    </joint>
-  <link name="camera_link"><inertial>
-      <mass value="1e-5" />
-      <origin xyz="0 0 0" rpy="0 0 0"/>
-      <inertia ixx="1e-6" ixy="0" ixz="0" iyy="1e-6" iyz="0" izz="1e-6" />
-    </inertial>
-  </link>
-  <link name="zed_camera_right_link">
-    <inertial>
-      <mass value="1e-5" />
-      <origin xyz="0 0 0" rpy="0 0 0"/>
-      <inertia ixx="1e-6" ixy="0" ixz="0" iyy="1e-6" iyz="0" izz="1e-6" />
-    </inertial>
-  </link>
-  <joint name="zed_camera_left_joint" type="fixed">
-    <origin xyz="0 0.06 0" rpy="0 0 0"/>
-    <parent link="zed_camera_link"/>
-    <child link="camera_link"/>
-    <axis xyz="0 0 1" />
-  </joint>
-  <joint name="zed_camera_right_joint" type="fixed">
-    <origin xyz="0 -0.06 0" rpy="0 0 0"/>
-    <parent link="zed_camera_link"/>
-    <child link="zed_camera_right_link"/>
-    <axis xyz="0 0 1" />
-  </joint>
+  <!-- ROS2 Control Section -->
   <ros2_control name="RaceCarHardware" type="system">
     <hardware>
       <plugin>gazebo_ros2_control/GazeboSystem</plugin>
     </hardware>
+    <!-- Steering joints -->
     <joint name="left_steering_hinge_joint">
       <command_interface name="position"/>
@@ -222,4 +64,10 @@
       <state_interface name="velocity"/>
     </joint>
+    <joint name="right_steering_hinge_joint">
+      <command_interface name="position"/>
+      <state_interface name="position"/>
+      <state_interface name="velocity"/>
+    </joint>
+    <!-- Rear wheels -->
     <joint name="left_rear_wheel_joint">
       <command_interface name="velocity"/>
@@ -232,4 +80,5 @@
       <state_interface name="velocity"/>
     </joint>
+    <!-- Front wheels (optional for Gazebo physics) -->
     <joint name="left_front_wheel_joint">
       <command_interface name="velocity"/>
@@ -242,11 +91,4 @@
       <state_interface name="velocity"/>
     </joint>
-    <joint name="right_steering_hinge_joint">
-      <command_interface name="position"/>
-      <state_interface name="position"/>
-      <state_interface name="velocity"/>
-    </joint>
   </ros2_control>
-  <xacro:include filename="$(find f1tenth_description)/urdf/racecar.gazebo" />
-  <xacro:include filename="$(find f1tenth_description)/urdf/materials.xacro" />
 </robot>
